Commit message: include script and reduce laserscanners

File: multi_jackal_description/urdf/OS1-64.urdf.xacro (robot description, xacro)
@@ -2,5 +2,6 @@
 <robot xmlns:xacro="http://www.ros.org/wiki/xacro" name="OS1-64">
   <xacro:property name="M_PI" value="3.1415926535897931" />
-  <xacro:macro name="OS1-64" params="*origin parent:=base_link name:=os1_sensor topic_points:=/os1_cloud_node/points topic_imu:=/os1_cloud_node/imu hz:=10 lasers:=16 samples:=512 min_range:=0.8 max_range:=60.0 noise:=0.008 min_angle:=-${M_PI} max_angle:=${M_PI} lidar_link:=os1_lidar imu_link:=os1_imu vfov_min:=-.29 vfov_max:=.29">
+  <!-- <xacro:macro name="OS1-64" params="*origin parent:=base_link name:=os1_sensor topic_points:=/os1_cloud_node/points topic_imu:=/os1_cloud_node/imu hz:=10 lasers:=16 samples:=512 min_range:=0.8 max_range:=60.0 noise:=0.008 min_angle:=-${M_PI} max_angle:=${M_PI} lidar_link:=os1_lidar imu_link:=os1_imu vfov_min:=-.29 vfov_max:=.29"> -->
+  <xacro:macro name="OS1-64" params="*origin parent:=base_link name:=os1_sensor topic_points:=/os1_cloud_node/points topic_imu:=/os1_cloud_node/imu hz:=10 lasers:=1 samples:=512 min_range:=0.8 max_range:=5.0 noise:=0.008 min_angle:=-${M_PI} max_angle:=${M_PI} lidar_link:=os1_lidar imu_link:=os1_imu vfov_min:=-.29 vfov_max:=.29">
     <joint name="${name}_mount_joint" type="fixed">
       <xacro:insert_block name="origin" />

File: multi_jackal_description/urdf/jackal_all.urdf.xacro (robot description, xacro)
@@ -302,8 +302,8 @@
       <origin xyz="0.0665 0 0.145"/>
   </joint>
-  <!-- <xacro:include filename="$(find multi_jackal_description)/urdf/OS1-64.urdf.xacro" />
+  <xacro:include filename="$(find multi_jackal_description)/urdf/OS1-64.urdf.xacro" />
   <OS1-64 parent="lidar_mounting_frame" name="os1" topic_imu="os1_cloud_node/imu" topic_points="os1_cloud_node/points">
     <origin xyz="0 0 0.035" rpy="0 0 0" />
-  </OS1-64> -->
+  </OS1-64>
   <!-- Bring in simulation data for Gazebo. -->
   <xacro:include filename="$(find multi_jackal_description)/urdf/jackal.gazebo" />

Commit message: Update OS1-64.urdf.xacro

File: multi_jackal_description/urdf/OS1-64.urdf.xacro (robot description, xacro)
@@ -3,5 +3,5 @@
   <xacro:property name="M_PI" value="3.1415926535897931" />
   <!-- <xacro:macro name="OS1-64" params="*origin parent:=base_link name:=os1_sensor topic_points:=/os1_cloud_node/points topic_imu:=/os1_cloud_node/imu hz:=10 lasers:=16 samples:=512 min_range:=0.8 max_range:=60.0 noise:=0.008 min_angle:=-${M_PI} max_angle:=${M_PI} lidar_link:=os1_lidar imu_link:=os1_imu vfov_min:=-.29 vfov_max:=.29"> -->
-  <xacro:macro name="OS1-64" params="*origin parent:=base_link name:=os1_sensor topic_points:=/os1_cloud_node/points topic_imu:=/os1_cloud_node/imu hz:=10 lasers:=1 samples:=512 min_range:=0.8 max_range:=5.0 noise:=0.008 min_angle:=-${M_PI} max_angle:=${M_PI} lidar_link:=os1_lidar imu_link:=os1_imu vfov_min:=-.29 vfov_max:=.29">
+  <xacro:macro name="OS1-64" params="*origin parent:=base_link name:=os1_sensor topic_points:=/os1_cloud_node/points topic_imu:=/os1_cloud_node/imu hz:=10 lasers:=1 samples:=512 min_range:=0.8 max_range:=5.0 noise:=0.008 min_angle:=-${M_PI} max_angle:=${M_PI} lidar_link:=os1_lidar imu_link:=os1_imu vfov_min:=-.0 vfov_max:=.0">
     <joint name="${name}_mount_joint" type="fixed">
       <xacro:insert_block name="origin" />
